File: HueTapSwitch(230V)/PCB/diyhue-IO.sch (EAGLE design)
At the start: 43 parts, among them IC1 MCP1825T-3302E/DC, X1 DG129-5.0, X2 DG129-5.0, X3 DG129-5.0

Commit message: changed Resistors on the inputs from 0805 to 1210
Parts:
- R10, R13, R14, R5, R6, R7, R8, R9: device rcl:R-EU_R0805W -> rcl:R-EU_R1210
Connections:
- net !RST: now also SV1.2
- net GND: now also SV1.1; no longer SV1.4, SV1.5
- net RX: now also SV1.4; no longer SV1.2
- net TX: now also SV1.5; no longer SV1.1
Other:
- note added: "+3V3"
- note added: "+5V"
- note added: "1.0"
- note added: "230V ~ Sicherung: 0.4A flink"
- note added: "3,3V (WiFi)"
- note added: "5V (Schaltregler)"
- note added: "Abstände"
- note added: "Entwurf/Prototyp 1"
- note added: "HV-HV"
- note added: "HV-LV"
- note added: "HV.###"
- note added: "Inspiriert vom Projekt "Open Source Blinds Controller" der In-Circuit GmbH Dresden (in-circuit.de)"
- note added: "Netzspannung"
- note added: "Revisionen"
- note added: "Supply-Netze"
- note added: "Versorgung"
- note added: "Überspannungskategorie: II"
- note added: "≥2,5mm Netz; 2,3mm abgesichert"
- note added: "≥5mm"
